File: soic8/soic8.sch (KiCad schematic (older format))
At the start: 3 parts, among them J1 Conn_01x04_Male, J2 Conn_01x04_Male, U1 ATSHA204_SOIC8

Commit message: Updated soic-8 with lib
Parts:
- removed J1, J2: Conn_01x04_Male, Connectors:1X04, symbol Connector:Conn_01x04_Male
- added J3: Conn_01x08_Male, DevPc:bb_2x4, symbol Connector:Conn_01x08_Male
- U1: footprint Silicon-Standard:SO08 -> DevPc:bb_2x4
Connections:
- wire segments 8 -> 16
Changed lines of the file:
@@
 F 0 "U1" H 5550 4410 45  0000 C CNN
 F 1 "ATSHA204_SOIC8" H 5550 4326 45  0000 C CNN
-F 2 "Silicon-Standard:SO08" H 5550 4250 20  0001 C CNN
+F 2 "DevPc:bb_2x4" H 5550 4250 20  0001 C CNN
 F 3 "" H 5550 3950 60  0001 C CNN
 F 4 "IC-11981" H 5550 4231 60  0000 C CNN "Field4"
 	1    5550 3950
 	1    0    0    -1
-$EndComp
-$Comp
-L Connector:Conn_01x04_Male J1
-U 1 1 5BC397F8
-P 4750 3950
-F 0 "J1" H 4856 4228 50  0000 C CNN
-F 1 "Conn_01x04_Male" H 4856 4137 50  0000 C CNN
-F 2 "Connectors:1X04" H 4750 3950 50  0001 C CNN
-F 3 "~" H 4750 3950 50  0001 C CNN
-	1    4750 3950
-	1    0    0    -1
-$EndComp
-$Comp
-L Connector:Conn_01x04_Male J2
-U 1 1 5BC39862
-P 6350 4050
-F 0 "J2" H 6323 3930 50  0000 R CNN
-F 1 "Conn_01x04_Male" H 6323 4021 50  0000 R CNN
-F 2 "Connectors:1X04" H 6350 4050 50  0001 C CNN
-F 3 "~" H 6350 4050 50  0001 C CNN
-	1    6350 4050
-	-1   0    0    1
 $EndComp
 Wire Wire Line
@@
 Wire Wire Line
 	4950 4150 5050 4150
+$Comp
+L Connector:Conn_01x08_Male J3
+U 1 1 5BC38A6E
+P 4750 4150
+F 0 "J3" H 4856 4628 50  0000 C CNN
+F 1 "Conn_01x08_Male" H 4856 4537 50  0000 C CNN
+F 2 "DevPc:bb_2x4" H 4750 4150 50  0001 C CNN
+F 3 "~" H 4750 4150 50  0001 C CNN
+	1    4750 4150
+	1    0    0    -1
+$EndComp
 Wire Wire Line
-	6050 3850 6150 3850
+	4950 4250 6200 4250
 Wire Wire Line
-	6150 3950 6050 3950
+	6200 4250 6200 4150
 Wire Wire Line
-	6050 4050 6150 4050
+	6050 4150 6200 4150
 Wire Wire Line
-	6150 4150 6050 4150
+	6250 4050 6250 4350
+Wire Wire Line
+	6250 4350 4950 4350
+Wire Wire Line
+	6050 4050 6250 4050
+Wire Wire Line
+	4950 4450 6350 4450
+Wire Wire Line
+	6350 4450 6350 3950
+Wire Wire Line
+	6050 3950 6350 3950
+Wire Wire Line
+	6450 3850 6450 4550
+Wire Wire Line
+	6450 4550 4950 4550
+Wire Wire Line
+	6050 3850 6450 3850
 $EndSCHEMATC

Commit message: Implemented library footprints on soic-8
Parts:
- removed J3: Conn_01x08_Male, DevPc:bb_2x4, symbol Connector:Conn_01x08_Male
- removed U1: ATSHA204_SOIC8, DevPc:bb_2x4, symbol SparkFun-IC-Special-Function:ATSHA204_SOIC8
- added J1: bb2x4, DevPc:bb_2x4, symbol DevPCBpackages:bb2x4
- added U1: u2x4, DevPc:soic-8, symbol DevPCBpackages:u2x4
Connections:
- wire segments 16 -> 8
Changed lines of the file:
@@
 $EndDescr
 $Comp
-L SparkFun-IC-Special-Function:ATSHA204_SOIC8 U1
-U 1 1 5BC39766
-P 5550 3950
-F 0 "U1" H 5550 4410 45  0000 C CNN
-F 1 "ATSHA204_SOIC8" H 5550 4326 45  0000 C CNN
-F 2 "DevPc:bb_2x4" H 5550 4250 20  0001 C CNN
-F 3 "" H 5550 3950 60  0001 C CNN
-F 4 "IC-11981" H 5550 4231 60  0000 C CNN "Field4"
-	1    5550 3950
+L DevPCBpackages:bb2x4 J1
+U 1 1 5BC44432
+P 6100 2550
+F 0 "J1" H 6125 2765 50  0000 C CNN
+F 1 "bb2x4" H 6125 2674 50  0000 C CNN
+F 2 "DevPc:bb_2x4" H 6100 2550 50  0001 C CNN
+F 3 "" H 6100 2550 50  0001 C CNN
+	1    6100 2550
+	1    0    0    -1
+$EndComp
+$Comp
+L DevPCBpackages:u2x4 U1
+U 1 1 5BC444C0
+P 6100 2500
+F 0 "U1" H 6100 2533 50  0000 C CNN
+F 1 "u2x4" H 6100 2000 50  0001 C CNN
+F 2 "DevPc:soic-8" H 6100 2500 50  0001 C CNN
+F 3 "" H 6100 2500 50  0001 C CNN
+	1    6100 2500
 	1    0    0    -1
 $EndComp
 Wire Wire Line
-	5050 3850 4950 3850
+	5650 2600 5850 2600
 Wire Wire Line
-	4950 3950 5050 3950
+	5850 2700 5650 2700
 Wire Wire Line
-	5050 4050 4950 4050
+	5650 2800 5850 2800
 Wire Wire Line
-	4950 4150 5050 4150
-$Comp
-L Connector:Conn_01x08_Male J3
-U 1 1 5BC38A6E
-P 4750 4150
-F 0 "J3" H 4856 4628 50  0000 C CNN
-F 1 "Conn_01x08_Male" H 4856 4537 50  0000 C CNN
-F 2 "DevPc:bb_2x4" H 4750 4150 50  0001 C CNN
-F 3 "~" H 4750 4150 50  0001 C CNN
-	1    4750 4150
-	1    0    0    -1
-$EndComp
+	5850 2900 5650 2900
 Wire Wire Line
-	4950 4250 6200 4250
+	6350 2900 6600 2900
 Wire Wire Line
-	6200 4250 6200 4150
+	6600 2800 6350 2800
 Wire Wire Line
-	6050 4150 6200 4150
+	6350 2700 6600 2700
 Wire Wire Line
-	6250 4050 6250 4350
-Wire Wire Line
-	6250 4350 4950 4350
-Wire Wire Line
-	6050 4050 6250 4050
-Wire Wire Line
-	4950 4450 6350 4450
-Wire Wire Line
-	6350 4450 6350 3950
-Wire Wire Line
-	6050 3950 6350 3950
-Wire Wire Line
-	6450 3850 6450 4550
-Wire Wire Line
-	6450 4550 4950 4550
-Wire Wire Line
-	6050 3850 6450 3850
+	6600 2600 6350 2600
 $EndSCHEMATC

Commit message: Added U2x8 and BB2x8 to lib
Parts:
- J1: symbol DevPCBpackages:bb2x4 -> DevPCB-packages:bb2x4
- U1: symbol DevPCBpackages:u2x4 -> DevPCB-packages:u2x4
Changed lines of the file:
@@
 $EndDescr
 $Comp
-L DevPCBpackages:bb2x4 J1
+L DevPCB-packages:bb2x4 J1
 U 1 1 5BC44432
 P 6100 2550
@@
 $EndComp
 $Comp
-L DevPCBpackages:u2x4 U1
+L DevPCB-packages:u2x4 U1
 U 1 1 5BC444C0
 P 6100 2500
