File: soic14/soic14.sch (KiCad schematic (older format))
At the start: 2 parts, among them J1 bb2x7, U1 u2x7

Commit message: SOIC14
Parts:
- added J?: bb2x7, DevPc:bb_2x7, symbol DevPCB-packages:bb2x7
- added U?: MSOP/TSSOP-14, DevPc:soic-14, symbol DevPCB-packages:u2x7
- U1: value u2x7 -> SOIC/SOP/SO-14
Connections:
- wire segments 14 -> 28
Changed lines of the file:
@@
 EESchema Schematic File Version 4
+LIBS:soic14-cache
 EELAYER 26 0
 EELAYER END
@@
 P 5150 2250
 F 0 "U1" H 5150 2250 50  0001 C CNN
-F 1 "u2x7" H 5150 1450 50  0001 C CNN
+F 1 "SOIC/SOP/SO-14" H 5150 1450 50  0001 C CNN
 F 2 "DevPc:soic-14" H 5150 2250 50  0001 C CNN
 F 3 "" H 5150 2250 50  0001 C CNN
@@
 Wire Wire Line
 	5400 2350 5600 2350
+$Comp
+L DevPCB-packages:bb2x7 J?
+U 1 1 5BCCCF9F
+P 5100 3400
+F 0 "J?" H 5100 3510 50  0001 C CNN
+F 1 "bb2x7" H 5100 2600 50  0001 C CNN
+F 2 "DevPc:bb_2x7" H 5100 3400 50  0001 C CNN
+F 3 "" H 5100 3400 50  0001 C CNN
+	1    5100 3400
+	1    0    0    -1
+$EndComp
+$Comp
+L DevPCB-packages:u2x7 U?
+U 1 1 5BCCCFA5
+P 5150 3350
+F 0 "U?" H 5150 3350 50  0001 C CNN
+F 1 "MSOP/TSSOP-14" H 5150 2550 50  0001 C CNN
+F 2 "DevPc:soic-14" H 5150 3350 50  0001 C CNN
+F 3 "" H 5150 3350 50  0001 C CNN
+	1    5150 3350
+	1    0    0    -1
+$EndComp
+Wire Wire Line
+	4900 3450 4650 3450
+Wire Wire Line
+	4650 3550 4900 3550
+Wire Wire Line
+	4900 3650 4650 3650
+Wire Wire Line
+	4650 3750 4900 3750
+Wire Wire Line
+	4900 3850 4650 3850
+Wire Wire Line
+	4650 3950 4900 3950
+Wire Wire Line
+	4900 4050 4650 4050
+Wire Wire Line
+	5400 4050 5600 4050
+Wire Wire Line
+	5600 3950 5400 3950
+Wire Wire Line
+	5400 3850 5600 3850
+Wire Wire Line
+	5600 3750 5400 3750
+Wire Wire Line
+	5400 3650 5600 3650
+Wire Wire Line
+	5600 3550 5400 3550
+Wire Wire Line
+	5400 3450 5600 3450
 $EndSCHEMATC
